Commit message: edits to yale hand files to make controllable version for Baxter

File: yale_openhand_models/urdf/wsn_model_t.xacro (robot description, xacro)
@@ -9,9 +9,17 @@
   <!--<xacro:include filename="gripper.gazebo" /-->
   <!-- xacro:include filename="$(find yale_openhand_models)/urdf/gripper.gazebo" / -->
+    <!-- wsn, copy and paste instead -->
+  <gazebo>
+    <plugin name="gazebo_ros_control" filename="libgazebo_ros_control.so">
+      <robotNamespace>gripper</robotNamespace>
+    </plugin>
+  </gazebo>
   <xacro:property name="controller" value="EffortJointInterface" />
   <xacro:macro name="trans" params="joint_name">
     <transmission name="${joint_name}_trans">
       <type>transmission_interface/SimpleTransmission</type>
-      <joint name="${joint_name}"/>
+      <joint name="${joint_name}">
+        <hardwareInterface>EffortJointInterface</hardwareInterface>
+       </joint>
       <actuator name="${joint_name}_actuator">
 	<hardwareInterface>${controller}</hardwareInterface>
@@ -28,6 +36,6 @@
     <inertial>
       <origin rpy="0 0 0" xyz="0 0 0" />
-      <mass value="1e-2" />
-      <inertia ixx="1e-3" ixy="0" ixz="0" iyy="1e-3" iyz="0" izz="1e-3" />
+      <mass value="1e-1" />
+      <inertia ixx="1e-2" ixy="0" ixz="0" iyy="1e-2" iyz="0" izz="1e-2" />
     </inertial>
     <visual>
@@ -115,6 +123,6 @@
       <inertial>
 	<origin rpy="0 0 0" xyz="0 0 0" />
-	<mass value="1e-2" />
-	<inertia ixx="1e-4" ixy="0" ixz="0" iyy="1e-4" iyz="0" izz="1e-4" />
+	<mass value="1e-1" />
+	<inertia ixx="1e-2" ixy="0" ixz="0" iyy="1e-2" iyz="0" izz="1e-2" />
       </inertial>
       <visual>
@@ -154,6 +162,6 @@
       <inertial>
 	<origin rpy="0 0 0" xyz="0 0 0" />
-	<mass value="1e-2" />
-	<inertia ixx="1e-4" ixy="0" ixz="0" iyy="1e-4" iyz="0" izz="1e-4" />
+	<mass value="1e-1" />
+	<inertia ixx="1e-2" ixy="0" ixz="0" iyy="1e-2" iyz="0" izz="1e-2" />
       </inertial>
       <visual>
@@ -184,3 +192,2 @@
   </xacro:macro>
   </robot>
-<!--/robot -->
